File: hardware/pole-node/pole-node.sch (KiCad schematic (older format))
At the start: 31 parts, among them J1 Anderson, J2 RJ45, J3 Conn_01x02, J4 Conn_01x03, J5 Conn_01x03, J6 Conn_01x03, U1 AP3211, U2 MAX485E, U3 MAX485E

Commit message: Update pole node to v1.1
This adds lots of TVS diode, more decoupling, bulk caps on 5v and 12v
lines. Also adds pass-through Anderson connector.
Parts:
- removed J3: Conn_01x02, Connector_PinHeader_2.54mm:PinHeader_1x02_P2.54mm_Vertical, symbol Connector_Generic:Conn_01x02
- added C10: .1uF, Capacitor_SMD:C_0603_1608Metric, symbol Device:C
- added C11, C12: 470uF, Capacitor_THT:CP_Radial_D10.0mm_P5.00mm, symbol Device:CP
- added D10, D11, D6, D7, D8, D9: D_TVS_DATA, Diode_SMD:D_SMA, symbol Device:D_TVS
- added D12: D_TVS_12V, Diode_SMD:D_SMB, symbol Device:D_TVS
- added D13, D14, D15: D_TVS_5V, Diode_SMD:D_SOD-523, symbol Device:D_TVS
- added J3: Conn_01x03, Connector_PinHeader_2.54mm:PinHeader_1x03_P2.54mm_Horizontal, symbol Connector_Generic:Conn_01x03
- added J7: Anderson, homebrew:Anderson_1336G1_right_angle_bottom_two, symbol Homebrew:Anderson_two_redblack_sink
- C2: MPN (none) -> CL10B122KB8NNNC
- D1: MPN (none) -> MBR230LSTR
- D2: MPN (none) -> 1N4148WS-7-F
- D3, D5: value D_TVS -> D_TVS_5V
- J1: footprint homebrew:Anderson_1337G3_right_angle_bottom_two -> homebrew:Anderson_1336G1_right_angle_bottom_two
- J2: MPN (none) -> 54601-908WPLF
- J4, J5, J6: footprint Connector_PinHeader_2.54mm:PinHeader_1x03_P2.54mm_Vertical -> Connector_PinHeader_2.54mm:PinHeader_1x03_P2.54mm_Horizontal
- L1: MPN (none) -> NR6028T6R0M
- U1: MPN (none) -> AP3211KTR-G1
- U2, U3: MPN (none) -> SP485ECN-L/TR
Connections:
- net +5V: now also C10.1, C12.1, D15.1 (A1)
- net GND: now also C10.2, C11.2, C12.2, D11.1 (A1), D12.2 (A2), D13.2 (A2), D14.2 (A2), D15.2 (A2), D6.1 (A1), D8.1 (A1), D9.1 (A1), J3.1 (Pin_1), J7.2
- net LED_1_A: now also D7.1 (A1), D8.2 (A2)
- net LED_1_B: now also D6.2 (A2), D7.2 (A2)
- net LED_1_OUT: now also D13.1 (A1), J3.2 (Pin_2)
- net LED_2_A: now also D10.1 (A1), D11.2 (A2)
- net LED_2_B: now also D10.2 (A2), D9.2 (A2)
- net LED_2_OUT: now also D14.1 (A1)
- net +12V: now reaches C1.1, J1.1, U1.4 (EN), U1.5 (IN)
- net +12V: now also C11.1, D12.1 (A1), J7.1
- no-connect marks 2 -> 3
Other:
- note removed: "TODO: check that pairs are correct"
- moved on the sheet: C1, C2, C3, C4, C5, C6, C7, D1, D2, D4, J1, L1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
