File: hardware/pole-node/pole-node.kicad_sch (KiCad schematic)
At the start: 46 parts, among them J1 Anderson_two_redblack_src, J2 RJ45, J3 Conn_01x03, J4 Conn_01x03, J5 Conn_01x03, J6 Conn_01x03, J7 Anderson_two_redblack_sink, U1 XL1509-5.0E1, U2 MAX485E, U3 MAX485E

Commit message: Fix pole-node v1.3 footprint for XL1509 SMPS
Parts:
- U1: footprint Package_SO:SOIC-8_5.23x5.23mm_P1.27mm -> Package_SO:SOIC-8_3.9x4.9mm_P1.27mm
Changed lines of the file:
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@@
       (effects (font (size 1.27 1.27)))
     )
-    (property "Footprint" "Package_SO:SOIC-8_5.23x5.23mm_P1.27mm" (at 105.41 27.94 0)
+    (property "Footprint" "Package_SO:SOIC-8_3.9x4.9mm_P1.27mm" (at 105.41 27.94 0)
       (effects (font (size 1.27 1.27)) hide)
     )
