File: hardware/colordance-brain/_autosave-colordance-brain.sch (KiCad schematic (older format))
At the start: 58 parts, among them J1 Anderson, J2 Conn_01x06, J3 Conn_01x03, J4 Conn_01x03, J5 Conn_01x03, J6 Conn_01x03, J7 Conn_01x06, J8 Conn_01x05, U1 AP3211, U2 Teensy4.1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

Commit message: Random hardware changes
Parts:
- H1, H2, H3, H4: symbol Homebrew:HOLE -> colordance-brain-rescue:HOLE-Homebrew-colordance-brain-rescue
- J1: symbol Homebrew:Anderson_two_redblack_src -> colordance-brain-rescue:Anderson_two_redblack_src-Homebrew-colordance-brain-rescue
- U1: symbol Homebrew:AP3211 -> colordance-brain-rescue:AP3211-Homebrew-colordance-brain-rescue
- U2: symbol teensy_library:Teensy4.1 -> colordance-brain-rescue:Teensy4.1-teensy_library-colordance-brain-rescue
Changed lines of the file:
@@
 $EndComp
 $Comp
-L Homebrew:AP3211 U1
+L colordance-brain-rescue:AP3211-Homebrew-colordance-brain-rescue U1
 U 1 1 5E594E3E
 P 2800 1400
@@
 	4400 1400 4700 1400
 $Comp
-L Homebrew:Anderson_two_redblack_src J1
+L colordance-brain-rescue:Anderson_two_redblack_src-Homebrew-colordance-brain-rescue J1
 U 1 1 5E5A16EF
 P 700 1300
@@
 $EndComp
 $Comp
-L Homebrew:HOLE H1
+L colordance-brain-rescue:HOLE-Homebrew-colordance-brain-rescue H1
 U 1 1 60A08675
 P 10450 8500
@@
 $EndComp
 $Comp
-L Homebrew:HOLE H2
+L colordance-brain-rescue:HOLE-Homebrew-colordance-brain-rescue H2
 U 1 1 60A09861
 P 10450 8750
@@
 $EndComp
 $Comp
-L Homebrew:HOLE H3
+L colordance-brain-rescue:HOLE-Homebrew-colordance-brain-rescue H3
 U 1 1 60A09A47
 P 10450 9000
@@
 $EndComp
 $Comp
-L Homebrew:HOLE H4
+L colordance-brain-rescue:HOLE-Homebrew-colordance-brain-rescue H4
 U 1 1 60A09CE3
 P 10450 9250
@@
 CS_AUDIO
 $Comp
-L teensy_library:Teensy4.1 U2
+L colordance-brain-rescue:Teensy4.1-teensy_library-colordance-brain-rescue U2
 U 1 1 607BEEC0
 P 11850 4450
