File: hardware/colordance-brain/rs422_output.sch (KiCad schematic (older format))
At the start: 24 parts, among them J2 RJ45, J3 RJ45, U3 AM26LS31x

Commit message: Colordance brain v1.0
Parts:
- removed D10, D11, D16, D17, D18, D6, D7, D8: D_TVS_DATA, Diode_SMD:D_SMA, symbol Device:D_TVS
- removed D13, D14, D5: D_TVS_5V, Diode_SMD:D_SOD-523, symbol Device:D_TVS
- added D23, D26, D27, D28, D29: D_TVS_DATA, Diode_SMD:D_SMB, symbol Device:D_TVS
- added D24, D25: D_TVS_5V, Diode_SMD:D_SMB, symbol Device:D_TVS
- C18: renamed from C5; value .1uF -> 0.1uF; footprint Capacitor_SMD:C_0603_1608Metric_Pad1.05x0.95mm_HandSolder -> Capacitor_SMD:C_0603_1608Metric
- C19: renamed from C6; value 100nF -> 0.1uF; footprint (none) -> Capacitor_SMD:C_0603_1608Metric
- C20: renamed from C7; value 100nF -> 0.1uF; footprint (none) -> Capacitor_SMD:C_0603_1608Metric
- C21: renamed from C8; value 100nF -> 0.1uF; footprint (none) -> Capacitor_SMD:C_0603_1608Metric
- C22: renamed from C9; value 100nF -> 0.1uF; footprint (none) -> Capacitor_SMD:C_0603_1608Metric
- D18: renamed from D3; footprint Diode_SMD:D_SOD-523 -> Diode_SMD:D_SMB; MPN CPDH5V0U -> SMBJ6.0CD-M3/H
- D19: value D_TVS_DATA -> D_TVS_5V; footprint Diode_SMD:D_SMA -> Diode_SMD:D_SMB; MPN 824501900 -> SMBJ6.0CD-M3/H
- D20, D21: footprint Diode_SMD:D_SMA -> Diode_SMD:D_SMB; MPN 824501900 -> SMBJ6.0CD-M3/H
- D22: renamed from D9; footprint Diode_SMD:D_SMA -> Diode_SMD:D_SMB; MPN 824501900 -> SMBJ6.0CD-M3/H
- J10: renamed from J3; MPN (none) -> 54601-908WPLF
- J9: renamed from J2; MPN (none) -> 54601-908WPLF
- U3: MPN (none) -> AM26LS31CDR
Connections:
- net GND: now also D20.1 (A1), D21.2 (A2), D23.1 (A1), D24.1 (A1), D25.1 (A1), D26.1 (A1), D27.2 (A2), D28.1 (A1), D29.1 (A1); no longer D21.1 (A1)
- net LED1_Y: now also D21.1 (A1)
- net LED1_Z: now also D20.2 (A2)
- net LED2_Y: now also D23.2 (A2)
- net LED3_Y: now also D29.2 (A2); no longer D20.1 (A1), D21.2 (A2)
- net LED3_Z: now also D28.2 (A2); no longer D19.2 (A2), D20.2 (A2)
- net LED4_Y: now also D27.1 (A1)
- net LED4_Z: now also D26.2 (A2)
- net PIR2: now also D19.2 (A2)
- net PIR3: now also D24.2 (A2)
- net PIR4: now also D25.2 (A2)

Commit message: Random hardware changes
Parts:
- U3: symbol Homebrew:AM26LS31x -> colordance-brain-rescue:AM26LS31x-Homebrew
Changed lines of the file:
@@
 	1150 2550 1550 2550
 $Comp
-L Homebrew:AM26LS31x U?
+L colordance-brain-rescue:AM26LS31x-Homebrew U?
 U 1 1 60932044
 P 1550 3400
