File: hardware/colordance-brain/colordance-brain.kicad_sch (KiCad schematic)
At the start: 58 parts

Commit message: colordance-brain v1.1
- Switch from SPI to serial-over-RS422 for communication with the
interface. Using the Teensy 4.1 as a SPI peripheral did not work. Using
RS422 will allow us to place the interface far away (e.g. 50ft) from the
brain.
- Also break out an extra serial port, e.g. for music playing?
- Change protection for most I/O pins to resistor + cap instead of TVS
diode
- Add a builtin button, for activating test modes
Parts:
- removed C13, C4: (no value), symbol Device:C
- removed D12, D13, D15, D16, D17, D5, D6, D7: (no value), symbol Device:D_TVS
- removed J2, J7: (no value), symbol Connector_Generic:Conn_01x06
- added C1, C15, C19: 0.1uF, Capacitor_SMD:C_0603_1608Metric, symbol Device:C
- added C20: 1300pF, Capacitor_SMD:C_0603_1608Metric, symbol Device:C
- added D11, D9: D_TVS_DATA, Diode_SMD:D_SMB, symbol Device:D_TVS
- added J2: Conn_01x04, Connector_PinHeader_2.54mm:PinHeader_1x04_P2.54mm_Horizontal, symbol Connector_Generic:Conn_01x04
- added J8: RJ45, Connector_RJ:RJ45_Amphenol_54602-x08_Horizontal, symbol Connector:RJ45
- added R12, R6, R7, R9: 1k, Resistor_SMD:R_0603_1608Metric, symbol Device:R
- added R13, R4, R5, R8: 100, Resistor_SMD:R_0603_1608Metric, symbol Device:R
- added R14: 120, Resistor_SMD:R_0603_1608Metric, symbol Device:R
- added SW1: SW_SPST, Button_Switch_THT:SW_PUSH_6mm, symbol Switch:SW_SPST
- added U5: ISL83490, Package_SO:SOIC-8_3.9x4.9mm_P1.27mm, symbol homebrew:ISL83490
- BT1: value (none) -> Battery_Cell; footprint (none) -> Battery:BatteryHolder_Keystone_3034_1x20mm
- C10: renamed from C11; value (none) -> 22nF; footprint (none) -> Capacitor_SMD:C_0603_1608Metric
- C11: renamed from C10; value (none) -> 22uF; footprint (none) -> Capacitor_SMD:C_0805_2012Metric
- C12, C9: value (none) -> 0.1uF; footprint (none) -> Capacitor_SMD:C_0603_1608Metric
- C13: renamed from C8; value (none) -> 0.1uF; footprint (none) -> Capacitor_SMD:C_0603_1608Metric
- C14: value (none) -> 470uF; footprint (none) -> Capacitor_THT:CP_Radial_D10.0mm_P5.00mm
- C16: renamed from C15; value (none) -> 0.1uF; footprint (none) -> Capacitor_SMD:C_0603_1608Metric
- C17: renamed from C16; value (none) -> 0.1uF; footprint (none) -> Capacitor_SMD:C_0603_1608Metric
- C18: renamed from C17; value (none) -> 0.1uF; footprint (none) -> Capacitor_SMD:C_0603_1608Metric
- C2: renamed from C1; value (none) -> 470uF; footprint (none) -> Capacitor_THT:CP_Radial_D10.0mm_P5.00mm
- C3: renamed from C2; value (none) -> 0.1uF; footprint (none) -> Capacitor_SMD:C_0603_1608Metric
- C4: renamed from C3; value (none) -> 0.1uF; footprint (none) -> Capacitor_SMD:C_0603_1608Metric
- C5: value (none) -> 10uF; footprint (none) -> Capacitor_SMD:C_0805_2012Metric
- C6: value (none) -> 22nF; footprint (none) -> Capacitor_SMD:C_0603_1608Metric
- C7: renamed from C33; value (none) -> 0.1uF; footprint (none) -> Capacitor_SMD:C_0603_1608Metric
- C8: renamed from C7; value (none) -> 10nF; footprint (none) -> Capacitor_SMD:C_0603_1608Metric
- D1: value (none) -> LED; footprint (none) -> LED_SMD:LED_0603_1608Metric
- D10, D8: value (none) -> D_TVS_DATA; footprint (none) -> Diode_SMD:D_SMB
- D2: value (none) -> D_TVS_12V; footprint (none) -> Diode_SMD:D_SMB
- D3, D4: value (none) -> D_TVS_5V; footprint (none) -> Diode_SMD:D_SMB
- D5: renamed from D9; value (none) -> SCHOTTKY; footprint (none) -> Diode_SMD:D_SOD-123
- D6: renamed from D11; value (none) -> D; footprint (none) -> Diode_SMD:D_SOD-323
- D7: renamed from D14; value (none) -> D_TVS_5V; footprint (none) -> Diode_SMD:D_SMB
- H1, H2, H3, H4: value (none) -> HOLE; footprint (none) -> homebrew:HOLE_5MM_#8
- J1: value (none) -> Anderson; footprint (none) -> homebrew:Anderson_1336G1_right_angle_bottom_two
- J3, J4: value (none) -> Conn_01x03; footprint (none) -> Connector_PinHeader_2.54mm:PinHeader_1x03_P2.54mm_Horizontal
- J5: renamed from J6; value (none) -> Conn_01x03; footprint (none) -> Connector_PinHeader_2.54mm:PinHeader_1x03_P2.54mm_Horizontal
- J6: renamed from J5; value (none) -> Conn_01x03; footprint (none) -> Connector_PinHeader_2.54mm:PinHeader_1x03_P2.54mm_Horizontal
- J7: renamed from J8; value (none) -> Conn_01x05; footprint (none) -> Connector_PinHeader_2.54mm:PinHeader_1x05_P2.54mm_Horizontal
- L1: value (none) -> 5.6uH; footprint (none) -> Inductor_SMD:L_Taiyo-Yuden_NR-60xx
- R1: value (none) -> 10k; footprint (none) -> Resistor_SMD:R_0603_1608Metric
- R10: renamed from R4; value (none) -> 11.5k; footprint (none) -> Resistor_SMD:R_0603_1608Metric
- R11: renamed from R5; value (none) -> 2.21k; footprint (none) -> Resistor_SMD:R_0603_1608Metric
- R2: value (none) -> 1.2M; footprint (none) -> Resistor_SMD:R_0805_2012Metric
- R3: value (none) -> 330k; footprint (none) -> Resistor_SMD:R_0603_1608Metric
- U1: renamed from U6; value (none) -> 74AHCT1G126; footprint (none) -> Package_TO_SOT_SMD:SOT-353_SC-70-5
- U2: renamed from U1; value (none) -> AP3211; footprint (none) -> Package_TO_SOT_SMD:SOT-23-6
- U3: renamed from U7; value (none) -> 74AHCT1G126; footprint (none) -> Package_TO_SOT_SMD:SOT-353_SC-70-5
- U4: renamed from U2; value (none) -> Teensy4.1; footprint (none) -> homebrew:Teensy41_stripped; MPN (none) -> PPPC241LFBN-RC
Connections:
- net +3V3: now also U4.15 (3V3), C15.1, C19.1, U5.1 (VCC)
- net +5V: now also C1.1, J2.4 (Pin_4)
- net BATT_DIV: now also R7.1; no longer C7.1, R2.2, R3.1
- net GND: now also D3.1 (A1), D4.1 (A1), C1.2, C15.2, C19.2, D11.1 (A1), D9.1 (A1), J2.1 (Pin_1), J8.3, J8.4, J8.5, J8.6, R9.2, U5.4 (GND); no longer D3.2 (A2), D4.2 (A2)
- net LOCAL_PIR0: now also R6.1; no longer J4.2 (Pin_2)
- net LOCAL_PIR1: now also R12.1; no longer J5.2 (Pin_2)
- net AUX_SERIAL_OUT: now reaches U4.10 (8_TX2_IN1)
- net AUX_SERIAL_OUT: now also D4.2 (A2), R8.1
- net INTERFACE_IN: now reaches U4.22 (30_CRX3)
- net INTERFACE_IN: now also U5.2 (RO)
- net INTERFACE_OUT: now reaches U4.23 (31_CTX3)
- net INTERFACE_OUT: now also U5.3 (DI)
- net AUX_SERIAL_IN: now reaches U4.9 (7_RX2_OUT1A)
- net AUX_SERIAL_IN: now also D3.2 (A2), R4.1
- net CONTROL_PANEL_LED renamed LOCAL_LED_1
- net CS_AUDIO renamed SW_BUILTIN
- net SW_BUILTIN: now also SW1.2 (B)
- net CS_CTRL: no longer names the net of U4.30 (38_CS1_IN1)
- net CS_CTRL: no longer D8.1 (A1)
- net MISO: no longer names the net of U4.31 (39_MISO1_OUT1A)
- net MOSI: no longer names the net of U4.18 (26_A12_MOSI1)
- net PODIUM_LED renamed LOCAL_LED_0
- net SCK: no longer names the net of U4.19 (27_A13_SCK1)
- net SCK: no longer D3.1 (A1)
- new net: C7.1, R2.2, R3.1, R7.2
- new net: J3.2 (Pin_2), R5.2
- new net: J6.2 (Pin_2), R13.2
- new net: J4.2 (Pin_2), R6.2
- new net: J5.2 (Pin_2), R12.2
- new net: R5.1, U1.4
- new net: R13.1, U3.4
- new net: R9.1, SW1.1 (A)
- new net: C20.1, R14.2
- new net: J2.2 (Pin_2), R4.2
- new net: J2.3 (Pin_3), R8.2
- new net INTERFACE_A: D8.1 (A1), J8.1, R14.1, U5.8 (A)
- new net INTERFACE_B: C20.2, D9.2 (A2), J8.2, U5.7 (B)
- new net INTERFACE_Y: D11.2 (A2), J8.8, U5.5 (Y)
- new net INTERFACE_Z: D10.1 (A1), J8.7, U5.6 (Z)
- no-connect marks 26 -> 25
Other:
- note removed: "SPI to audio"
- note removed: "SPI to control surface"
- moved on the sheet: C10, C6

Commit message: Move power supply to subsheet
Parts:
- removed C11: 22uF, Capacitor_SMD:C_0805_2012Metric, symbol Device:C
- removed C12: 0.1uF, Capacitor_SMD:C_0603_1608Metric, symbol Device:C
- removed C14, C2: 470uF, Capacitor_THT:CP_Radial_D10.0mm_P5.00mm, symbol Device:CP
- removed C5: 10uF, Capacitor_SMD:C_0805_2012Metric, symbol Device:C
- removed C8: 10nF, Capacitor_SMD:C_0603_1608Metric, symbol Device:C
- removed D2: D_TVS_12V, Diode_SMD:D_SMB, symbol Device:D_TVS
- removed D5: SCHOTTKY, Diode_SMD:D_SOD-123, symbol Device:D
- removed D6: D, Diode_SMD:D_SOD-323, symbol Device:D
- removed D7: D_TVS_5V, Diode_SMD:D_SMB, symbol Device:D_TVS
- removed J1: Anderson, homebrew:Anderson_1336G1_right_angle_bottom_two, symbol colordance-brain-rescue:Anderson_two_redblack_src-Homebrew
- removed L1: 5.6uH, Inductor_SMD:L_Taiyo-Yuden_NR-60xx, symbol Device:L
- removed R10: 11.5k, Resistor_SMD:R_0603_1608Metric, symbol Device:R
- removed R11: 2.21k, Resistor_SMD:R_0603_1608Metric, symbol Device:R
- removed U2: AP3211, Package_TO_SOT_SMD:SOT-23-6, symbol colordance-brain-rescue:AP3211-Homebrew
- renumbered C16 to C10, C17 to C11, C18 to C12, C19 to C13, C20 to C14, C3 to C2, C4 to C3, C6 to C4, C7 to C5, C9 to C6, C10 to C7, C13 to C8, C15 to C9, D3 to D2, D4 to D3, D8 to D4, D9 to D5, D10 to D6, D11 to D7, J2 to J1, J3 to J2, J4 to J3, J5 to J4, J6 to J5, J7 to J6, J8 to J7, R12 to R10, R13 to R11, R14 to R12, U3 to U2, U4 to U3, U5 to U4
Other:
- added sheet 5v_smps (5v_smps.kicad_sch)
- note removed: "Power"
- moved on the sheet: C5, D1, R1, R2, R3, R7, R9, SW1

Commit message: Start updating brain for v1.2
Parts:
- added C36: 0.1uF, Capacitor_SMD:C_0603_1608Metric, symbol Device:C
- added C37: 22nF, Capacitor_SMD:C_0603_1608Metric, symbol Device:C
- added C38: 470uF, Capacitor_THT:CP_Radial_D10.0mm_P5.00mm, symbol Device:CP
- added J15: Conn_01x03, Connector_PinHeader_2.54mm:PinHeader_1x03_P2.54mm_Horizontal, symbol Connector_Generic:Conn_01x03
- added R27: 1k, Resistor_SMD:R_0603_1608Metric, symbol Device:R
- H1, H2, H3, H4: footprint homebrew:HOLE_5MM_#8 -> Homebrew:HOLE_5MM_#8
- U3: footprint homebrew:Teensy41_stripped -> Homebrew:Teensy41_stripped
Connections:
- net +3V3: now also C38.1
- net +5V: now also C36.1, J15.3 (Pin_3)
- net GND: now also C36.2, C37.2, C38.2, J15.1 (Pin_1)
- net INTERFACE_IN: now also U3.17 (25_A11_RX6_SDA2); no longer U3.22 (30_CRX3)
- net INTERFACE_OUT: now also U3.16 (24_A10_TX6_SCL2); no longer U3.23 (31_CTX3)
- net LOCAL_LED_0: now also U3.23 (31_CTX3); no longer U3.17 (25_A11_RX6_SDA2)
- net LOCAL_LED_1: now also U3.22 (30_CRX3); no longer U3.16 (24_A10_TX6_SCL2)
- net LOCAL_PIR2: now reaches U3.19 (27_A13_SCK1)
- net LOCAL_PIR2: now also C37.1, R27.1
- new net: J15.2 (Pin_2), R27.2
- no-connect marks 25 -> 24
Other:
- moved on the sheet: C6, C7, J4, J6, R10

Commit message: Update colordance-brain schematic for v1.3: JLC assembly
Parts:
- added R25: 2k2, Resistor_SMD:R_0603_1608Metric, symbol Device:R
- added R26: 3k3, Resistor_SMD:R_0603_1608Metric, symbol Device:R
- C1, C10, C11, C12, C13, C2, C3, C36, C5, C6, C8, C9: value 0.1uF -> 100nF; footprint Capacitor_SMD:C_0603_1608Metric -> Capacitor_SMD:C_0402_1005Metric; LCSC (none) -> C307331
- C14: LCSC (none) -> C1595
- C37, C4, C7: LCSC (none) -> C21122
- D1: LCSC (none) -> C2286
- D2, D3, D4, D5, D6, D7: LCSC (none) -> C78395
- H1, H2, H3, H4: symbol colordance-brain-rescue:HOLE-Homebrew -> Homebrew:HOLE
- R1: LCSC (none) -> C25804
- R10, R27, R6, R7, R9: LCSC (none) -> C21190
- R11, R4, R5, R8: value 100 -> 470; LCSC (none) -> C23179
- R12: LCSC (none) -> C22787
- R2: value 1.2M -> 120k; footprint Resistor_SMD:R_0805_2012Metric -> Resistor_SMD:R_0603_1608Metric; LCSC (none) -> C25808
- R3: value 330k -> 33k; LCSC (none) -> C4216
- U1, U2: footprint Package_TO_SOT_SMD:SOT-353_SC-70-5 -> Package_TO_SOT_SMD:SOT-23-5; LCSC (none) -> C163712
- U4: value ISL83490 -> MAX488E; symbol homebrew:ISL83490 -> Homebrew:ISL83490; LCSC (none) -> C10919; MPN ISL83490IBZ-T -> (none)
Connections:
- net GND: now also R26.2
- net INTERFACE_IN: now also R25.2, R26.1; no longer U4.2 (RO)
- new net: R25.1, U4.2 (RO)

Commit message: Update colordance-brain to 1.3: JLC assembly (completed)
Connections:
- net +3V3: no longer C13.1, U4.1 (VCC)
- net +5V: now also C13.1, U4.1 (VCC)
Changed lines of the file:
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@@
   (junction (at 52.07 93.98) (diameter 0) (color 0 0 0 0)
   )
+  (junction (at 448.31 35.56) (diameter 0) (color 0 0 0 0)
+  )
   (junction (at 44.45 238.76) (diameter 0) (color 0 0 0 0)
   )
@@
   (junction (at 284.48 156.21) (diameter 0) (color 0 0 0 0)
   )
-  (junction (at 434.34 35.56) (diameter 0) (color 0 0 0 0)
-  )
   (junction (at 137.16 255.27) (diameter 0) (color 0 0 0 0)
   )
@@
     )
   )
-  (symbol (lib_id "power:+3V3") (at 434.34 35.56 0) (unit 1)
-    (in_bom yes) (on_board yes) (dnp no)
-    (property "Reference" "#PWR037" (at 434.34 39.37 0)
-      (effects (font (size 1.27 1.27)) hide)
-    )
-    (property "Value" "+3V3" (at 434.721 31.1658 0)
-      (effects (font (size 1.27 1.27)))
-    )
-    (property "Footprint" "" (at 434.34 35.56 0)
-      (effects (font (size 1.27 1.27)) hide)
-    )
-    (property "Datasheet" "" (at 434.34 35.56 0)
-      (effects (font (size 1.27 1.27)) hide)
-    )
-    (pin "1")
-    (instances
-      (project "colordance-brain"
-        (path "/67fde712-c227-4662-83fd-8edd7efd58d3"
-          (reference "#PWR037") (unit 1)
-        )
-      )
-    )
-  )
   (symbol (lib_id "power:GND") (at 469.9 59.69 0) (unit 1)
     (in_bom yes) (on_board yes) (dnp no) (fields_autoplaced)
@@
         )
       )
+    )
+  )
+  (symbol (lib_id "power:+5V") (at 448.31 35.56 0) (unit 1)
+    (in_bom yes) (on_board yes) (dnp no)
+    (property "Reference" "#PWR037" (at 448.31 39.37 0)
+      (effects (font (size 1.27 1.27)) hide)
+    )
+    (property "Value" "+5V" (at 448.691 31.1658 0)
+      (effects (font (size 1.27 1.27)))
+    )
+    (property "Footprint" "" (at 448.31 35.56 0)
+      (effects (font (size 1.27 1.27)) hide)
+    )
+    (property "Datasheet" "" (at 448.31 35.56 0)
+      (effects (font (size 1.27 1.27)) hide)
+    )
+    (pin "1")
+    (instances
+      (project "colordance-brain"
+        (path "/67fde712-c227-4662-83fd-8edd7efd58d3"
+          (reference "#PWR037") (unit 1)
+        )
+      )
