File: hardware/colordance-brain/rs422_output.kicad_sch (KiCad schematic)
At the start: 20 parts

Commit message: colordance-brain v1.1
- Switch from SPI to serial-over-RS422 for communication with the
interface. Using the Teensy 4.1 as a SPI peripheral did not work. Using
RS422 will allow us to place the interface far away (e.g. 50ft) from the
brain.
- Also break out an extra serial port, e.g. for music playing?
- Change protection for most I/O pins to resistor + cap instead of TVS
diode
- Add a builtin button, for activating test modes
Parts:
- removed C? (x2): (no value), symbol Device:C
- removed D? (x4): (no value), symbol Device:D_TVS
- added C24, C25: 22nF, Capacitor_SMD:C_0603_1608Metric, symbol Device:C
- added R15, R16, R17, R18: 1k, Resistor_SMD:R_0603_1608Metric, symbol Device:R
- C21: renamed from C?; value (none) -> 0.1uF; footprint (none) -> Capacitor_SMD:C_0603_1608Metric
- C22, C23: renamed from C?; value (none) -> 22nF; footprint (none) -> Capacitor_SMD:C_0603_1608Metric
- D12, D13, D14, D15, D16, D17, D18, D19: renamed from D?; value (none) -> D_TVS_DATA; footprint (none) -> Diode_SMD:D_SMB
- J10, J9: renamed from J?; value (none) -> RJ45; footprint (none) -> Connector_RJ:RJ45_Amphenol_54602-x08_Horizontal
- U6: renamed from U?; value (none) -> AM26LS31x; footprint (none) -> Package_SO:SOIC-16_3.9x9.9mm_P1.27mm
Connections:
- net GND: now also C24.2, C25.2
- net PIR1: now also R15.1; no longer J9.6
- net PIR2: now also R16.1; no longer J9.5
- net PIR3: now also C24.1, R17.1; no longer J10.6
- net PIR4: now also C25.1, R18.1; no longer J10.5
- new net: J9.5, R16.2
- new net: J9.6, R15.2
- new net: J10.5, R18.2
- new net: J10.6, R17.2
Other:
- moved on the sheet: C22, C23

Commit message: Move power supply to subsheet
Parts:
- renumbered C21 to C15, C22 to C16, C23 to C17, C24 to C18, C25 to C19, D14 to D10, D15 to D11, D16 to D12, D17 to D13, D18 to D14, D19 to D15, D12 to D8, D13 to D9, J9 to J8, J10 to J9, R15 to R13, R16 to R14, R17 to R15, R18 to R16, U6 to U5

Commit message: Update colordance-brain PCB files to KiCAD 7
Parts:
- U5: LCSC (none) -> C6179

Commit message: Update colordance-brain schematic for v1.3: JLC assembly
Parts:
- C15: value 0.1uF -> 100nF; footprint Capacitor_SMD:C_0603_1608Metric -> Capacitor_SMD:C_0402_1005Metric; LCSC (none) -> C307331
- C16, C17, C18, C19: LCSC (none) -> C21122
- D10, D11, D12, D13, D14, D15, D8, D9: LCSC (none) -> C78395
- R13, R14, R15, R16: LCSC (none) -> C21190
- U5: symbol colordance-brain-rescue:AM26LS31x-Homebrew -> Homebrew:AM26LS31x
Changed lines of the file:
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@@
       (effects (font (size 1.27 1.27)) hide)
     )
-    (property "LCSC" "" (at 124.46 50.8 0)
+    (property "LCSC" "C78395" (at 124.46 50.8 0)
       (effects (font (size 1.27 1.27)) hide)
     )
@@
       (effects (font (size 1.27 1.27)) hide)
     )
-    (property "LCSC" "" (at 118.11 85.09 0)
+    (property "LCSC" "C78395" (at 118.11 85.09 0)
       (effects (font (size 1.27 1.27)) hide)
     )
@@
       (effects (font (size 1.27 1.27)) hide)
     )
-    (property "LCSC" "" (at 118.11 105.41 0)
+    (property "LCSC" "C78395" (at 118.11 105.41 0)
       (effects (font (size 1.27 1.27)) hide)
     )
@@
       (effects (font (size 1.27 1.27)) hide)
     )
-    (property "LCSC" "" (at 222.25 50.8 0)
+    (property "LCSC" "C78395" (at 222.25 50.8 0)
       (effects (font (size 1.27 1.27)) hide)
     )
@@
       (effects (font (size 1.27 1.27)) hide)
     )
-    (property "LCSC" "" (at 222.25 30.48 0)
+    (property "LCSC" "C78395" (at 222.25 30.48 0)
       (effects (font (size 1.27 1.27)) hide)
     )
@@
       (effects (font (size 1.27 1.27)) hide)
     )
-    (property "LCSC" "" (at 215.9 85.09 0)
+    (property "LCSC" "C78395" (at 215.9 85.09 0)
       (effects (font (size 1.27 1.27)) hide)
     )
@@
       (effects (font (size 1.27 1.27)) hide)
     )
-    (property "LCSC" "" (at 215.9 105.41 0)
+    (property "LCSC" "C78395" (at 215.9 105.41 0)
       (effects (font (size 1.27 1.27)) hide)
     )
@@
       (effects (font (size 1.27 1.27)) (justify left))
     )
-    (property "Value" "0.1uF" (at 57.531 67.183 0)
-      (effects (font (size 1.27 1.27)) (justify left))
-    )
-    (property "Footprint" "Capacitor_SMD:C_0603_1608Metric" (at 55.5752 69.85 0)
+    (property "Value" "100nF" (at 57.531 67.183 0)
+      (effects (font (size 1.27 1.27)) (justify left))
+    )
+    (property "Footprint" "Capacitor_SMD:C_0402_1005Metric" (at 55.5752 69.85 0)
       (effects (font (size 1.27 1.27)) hide)
     )
@@
       (effects (font (size 1.27 1.27)) hide)
     )
-    (property "LCSC" "" (at 54.61 66.04 0)
+    (property "LCSC" "C307331" (at 54.61 66.04 0)
       (effects (font (size 1.27 1.27)) hide)
     )
@@
     )
   )
-  (symbol (lib_id "colordance-brain-rescue:AM26LS31x-Homebrew") (at 39.37 86.36 0) (unit 1)
+  (symbol (lib_id "Homebrew:AM26LS31x") (at 39.37 86.36 0) (unit 1)
     (in_bom yes) (on_board yes) (dnp no)
     (property "Reference" "U5" (at 46.99 107.95 0)
@@
       (effects (font (size 1.27 1.27)) hide)
     )
-    (property "LCSC" "" (at 115.57 68.58 0)
+    (property "LCSC" "C21122" (at 115.57 68.58 0)
       (effects (font (size 1.27 1.27)) hide)
     )
@@
       (effects (font (size 1.27 1.27)) hide)
     )
-    (property "LCSC" "" (at 96.52 66.04 0)
+    (property "LCSC" "C21122" (at 96.52 66.04 0)
       (effects (font (size 1.27 1.27)) hide)
     )
@@
       (effects (font (size 1.27 1.27)) hide)
     )
-    (property "LCSC" "" (at 124.46 30.48 0)
+    (property "LCSC" "C78395" (at 124.46 30.48 0)
       (effects (font (size 1.27 1.27)) hide)
     )
@@
       (effects (font (size 1.27 1.27)) hide)
     )
-    (property "LCSC" "" (at 100.33 62.23 0)
+    (property "LCSC" "C21190" (at 100.33 62.23 0)
       (effects (font (size 1.27 1.27)) hide)
     )
@@
       (effects (font (size 1.27 1.27)) hide)
     )
-    (property "LCSC" "" (at 198.12 62.23 0)
+    (property "LCSC" "C21190" (at 198.12 62.23 0)
       (effects (font (size 1.27 1.27)) hide)
     )
@@
       (effects (font (size 1.27 1.27)) hide)
     )
-    (property "LCSC" "" (at 213.36 68.58 0)
+    (property "LCSC" "C21122" (at 213.36 68.58 0)
       (effects (font (size 1.27 1.27)) hide)
     )
@@
       (effects (font (size 1.27 1.27)) hide)
     )
-    (property "LCSC" "" (at 194.31 66.04 0)
+    (property "LCSC" "C21122" (at 194.31 66.04 0)
       (effects (font (size 1.27 1.27)) hide)
     )
@@
       (effects (font (size 1.27 1.27)) hide)
     )
-    (property "LCSC" "" (at 217.17 64.77 0)
+    (property "LCSC" "C21190" (at 217.17 64.77 0)
       (effects (font (size 1.27 1.27)) hide)
     )
@@
       (effects (font (size 1.27 1.27)) hide)
     )
-    (property "LCSC" "" (at 119.38 64.77 0)
-      (effects (font (size 1.27 1.27)) hide)
-    )
+    (property "LCSC" "C21190" (at 119.38 64.77 0)
+      (effects (font (size 1.27 1.27)) hide)
+    )
