File: hardware/interface-brain/5v_smps.kicad_sch (KiCad schematic)
At the start: 17 parts, among them J1 Anderson, U5 AP3211

Commit message: interface-brain v1.1:
- Switch to serial-over-RS422 for comms with colordance-brain
- Add 12v supply + 5V SMPS
Parts:
- J1: footprint homebrew:Anderson_1336G1_right_angle_bottom_two -> Homebrew:Anderson_1336G1_right_angle_bottom_two
Changed lines of the file:
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@@
       (effects (font (size 1.524 1.524)))
     )
-    (property "Footprint" "homebrew:Anderson_1336G1_right_angle_bottom_two" (id 2) (at 33.02 50.8 0)
+    (property "Footprint" "Homebrew:Anderson_1336G1_right_angle_bottom_two" (id 2) (at 33.02 50.8 0)
       (effects (font (size 1.524 1.524)) hide)
     )
