File: hardware/interface-brain/interface-brain.kicad_pcb (KiCad board)
At the start: 2 copper layers, 154 parts, among them J1 Conn_01x06, J10 Conn_01x03, J11 Conn_01x03, J12 Conn_01x03, J13 Conn_01x03, J14 Conn_01x03, J15 Conn_01x03, J16 Conn_01x03, J17 Conn_01x03, J18 Conn_01x02, J19 Conn_01x02, J2 Conn_01x03, J20 Conn_01x02, J21 Conn_01x02, J22 Conn_01x03, J23 Conn_01x03, J24 Conn_01x03, J25 Conn_01x03, J26 Conn_01x02, J27 Conn_01x02, J28 Conn_01x02, J29 Conn_01x02, J3 Conn_01x03, J30 Conn_01x03, J31 Conn_01x03, J32 Conn_01x03, J33 Conn_01x03, J34 Conn_01x02, J35 Conn_01x02, J36 Conn_01x02, J37 Conn_01x02, J38 Conn_01x02, J39 Conn_01x02, J4 Conn_01x03, J5 Conn_01x03, J6 Conn_01x03, J7 Conn_01x03, J8 Conn_01x03, J9 Conn_01x03, U3 Teensy4.1

Commit message: Continue interface brain layout
Parts:
- added H1: MountingHole, MountingHole:MountingHole_3.2mm_M3, F.Cu at (142.0, 35.0)
- added H2: MountingHole, MountingHole:MountingHole_3.2mm_M3, F.Cu at (35.0, 119.0)
- added H3: MountingHole, MountingHole:MountingHole_3.2mm_M3, F.Cu at (142.7, 119.0)
- added H4: MountingHole, MountingHole:MountingHole_3.2mm_M3, F.Cu at (49.0, 35.0)
- added U1: SN74ACT244PWR, Package_SO:TSSOP-20_4.4x6.5mm_P0.65mm, B.Cu at (133.2, 46.0)
- added U2: SN74ACT244PWR, Package_SO:TSSOP-20_4.4x6.5mm_P0.65mm, B.Cu at (134.9, 88.2)
- C1, C10, C11, C12, C13, C14, C15, C16, C17, C18, C19, C2, C20, C21, C22, C23, C24, C25, C26, C27, C28, C29, C3, C30, C31, C32, C33, C34, C35, C36, C37, C38, C39, C4, C40, C41, C42, C43, C44, C45, C46, C47, C48, C49, C5, C50, C51, C52, C53, C6, C8, C9, D1, D2, D3, D4, D5, D6, R1, R10, R11, R12, R13, R14, R15, R16, R17, R18, R19, R2, R20, R21, R22, R23, R24, R25, R26, R27, R28, R29, R3, R30, R31, R32, R33, R34, R35, R36, R37, R38, R39, R4, R40, R41, R42, R43, R44, R45, R46, R47, R48, R49, R5, R50, R51, R52, R53, R54, R55, R6, R7, R8, R9: moved to B.Cu
- moved C4 248.7 mm to (27.6, 100.0), turned to 180 degrees
- moved R29 242.9 mm to (39.9, 94.1)
- moved R27 240.6 mm to (39.0, 53.1), turned to 90 degrees
- moved R55 238.2 mm to (45.4, 115.0)
- moved J39 235.7 mm to (44.0, 119.0), turned to 90 degrees
- moved R13 226.7 mm to (57.6, 79.9), turned to 90 degrees
- moved R21 223.8 mm to (27.6, 80.0), turned to 90 degrees
- moved C2 222.8 mm to (27.6, 57.9), turned to 180 degrees
- moved J9 218.3 mm to (55.0, 98.0), turned to 90 degrees
- moved C10 217.6 mm to (57.6, 75.1), turned to 180 degrees
- moved R28 217.3 mm to (39.8, 74.9)
- moved R9 216.6 mm to (57.6, 37.8), turned to 90 degrees
- moved J7 215.4 mm to (55.0, 56.0), turned to 90 degrees
- moved C8 215.0 mm to (57.5, 33.1), turned to 180 degrees
- moved R54 214.6 mm to (26.4, 115.0)
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Connections:
- J10 pad 2: /LED9_OUT -> /LED3_OUT
- J11 pad 2: /LED10_OUT -> /LED7_OUT
- J13 pad 2: /LED12_OUT -> /LED15_OUT
- J14 pad 2: /LED13_OUT -> /LED4_OUT
- J15 pad 2: /LED14_OUT -> /LED8_OUT
- J16 pad 2: /LED15_OUT -> /LED12_OUT
- J3 pad 2: /LED2_OUT -> /LED5_OUT
- J4 pad 2: /LED3_OUT -> /LED9_OUT
- J5 pad 2: /LED4_OUT -> /LED13_OUT
- J6 pad 2: /LED5_OUT -> /LED2_OUT
- J8 pad 2: /LED7_OUT -> /LED10_OUT
- J9 pad 2: /LED8_OUT -> /LED14_OUT
- U3 pad 21: /BUTTON_6 -> /BUTTON_3
- U3 pad 6: /BUTTON_3 -> /BUTTON_6
Routing:
- net /BUTTON_5: track 0.00 -> 138.8 mm, vias 0 -> 2
- net /BUTTON_9: track 0.00 -> 131.0 mm, vias 0 -> 2
- net /BUTTON_1: track 0.00 -> 129.8 mm, vias 0 -> 2
- net /BUTTON_2: track 0.00 -> 114.2 mm, vias 0 -> 1
- net Net-(R21-Pad1): track 0.00 -> 114.0 mm, vias 0 -> 2
- net Net-(R23-Pad1): track 0.00 -> 113.4 mm, vias 0 -> 2
- net Net-(R17-Pad1): track 0.00 -> 112.1 mm, vias 0 -> 2
- net Net-(U1-Pad9): track 0.00 -> 112.0 mm, vias 0 -> 2
- net /ANALOG_1: track 0.00 -> 87.4 mm, vias 0 -> 2
- net Net-(U2-Pad14): track 0.00 -> 84.2 mm, vias 0 -> 2
- net Net-(R15-Pad1): track 0.00 -> 83.4 mm, vias 0 -> 2
- net /BUTTON_6: track 0.00 -> 82.5 mm, vias 0 -> 1
- net Net-(R9-Pad1): track 0.00 -> 82.1 mm, vias 0 -> 2
- net Net-(U1-Pad7): track 0.00 -> 82.0 mm, vias 0 -> 2
- net Net-(R22-Pad1): track 0.00 -> 54.6 mm, vias 0 -> 2
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Other:
- board outline added: 144 x 105 mm

Commit message: Interface brain layout almost done
Parts:
- D6: moved to F.Cu
- moved R42 156.0 mm to (67.4, 116.8), turned to 0 degrees
- moved C48 155.3 mm to (66.5, 120.8)
- moved R50 152.0 mm to (67.4, 115.0), turned to 0 degrees
- moved R51 151.8 mm to (88.8, 115.0), turned to 0 degrees
- moved R43 147.0 mm to (88.8, 116.8), turned to 0 degrees
- moved C49 137.8 mm to (88.0, 120.8)
- moved R52 134.3 mm to (109.8, 115.0), turned to 0 degrees
- moved D1 133.1 mm to (150.8, 105.8), turned to 90 degrees
- moved C50 125.0 mm to (109.1, 120.8)
- moved R44 122.5 mm to (109.8, 116.8), turned to 0 degrees
- moved D4 120.1 mm to (159.8, 105.8), turned to 90 degrees
- moved D2 118.3 mm to (153.1, 105.8), turned to 90 degrees
- moved D5 118.1 mm to (157.6, 105.8), turned to 90 degrees
- moved D3 111.9 mm to (155.4, 105.8), turned to 90 degrees
- moved C51 108.4 mm to (132.0, 120.8)
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Connections:
- U3 pad 10: /LED16_SIG -> /LED4_SIG
- U3 pad 11: /LED14_SIG -> /LED13_SIG
- U3 pad 16: /LED3_SIG -> /LED14_SIG
- U3 pad 17: /LED4_SIG -> /LED15_SIG
- U3 pad 18: /ANALOG_7 -> /ANALOG_5
- U3 pad 20: /BUTTON_5 -> /BUTTON_3
- U3 pad 21: /BUTTON_3 -> /BUTTON_4
- U3 pad 24: /LED15_SIG -> /LED16_SIG
- U3 pad 26: /BUTTON_10 -> /BUTTON_14
- U3 pad 31: /ANALOG_2 -> /ANALOG_7
- U3 pad 36: /LED7_SIG -> /LED12_SIG
- U3 pad 37: /LED8_SIG -> /LED11_SIG
- U3 pad 40: /LED6_SIG -> /LED8_SIG
- U3 pad 41: /LED5_SIG -> /LED7_SIG
- U3 pad 42: /ANALOG_5 -> /ANALOG_2
- U3 pad 44: /LED11_SIG -> /LED6_SIG
- U3 pad 45: /LED12_SIG -> /LED5_SIG
- U3 pad 7: /BUTTON_4 -> /BUTTON_5
- U3 pad 8: /LED13_SIG -> /LED3_SIG
- U3 pad 9: /BUTTON_14 -> /BUTTON_10
Routing:
- net /BUTTON_13: track 0.00 -> 174.0 mm, vias 0 -> 3
- net /BUTTON_11: track 0.00 -> 144.5 mm, vias 0 -> 1
- net /BUTTON_14: track 0.00 -> 142.4 mm, vias 0 -> 2
- net /ANALOG_6: track 0.00 -> 139.6 mm, vias 0 -> 1
- net /BUTTON_3: track 0.00 -> 122.2 mm, vias 0 -> 2
- net /BUTTON_4: track 0.00 -> 118.9 mm, vias 0 -> 2
- net /ANALOG_5: track 0.00 -> 118.2 mm, vias 0 -> 2
- net /BUTTON_7: track 0.00 -> 94.4 mm, vias 0 -> 2
- net /ANALOG_7: track 0.00 -> 90.9 mm, vias 0 -> 1
- net /BUTTON_8: track 0.00 -> 81.7 mm, vias 0 -> 1
- net /BUTTON_12: track 0.00 -> 77.4 mm, vias 0 -> 2
- net /LED9_SIG: track 0.00 -> 61.1 mm, vias 0 -> 3
- net /BUTTON_10: track 0.00 -> 57.3 mm, vias 0 -> 2
- net /LED10_SIG: track 0.00 -> 57.1 mm, vias 0 -> 3
- net /ANALOG_4: track 0.00 -> 55.7 mm, vias 0 -> 2
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- added copper zone on B.Cu, net GND
- added copper zone on F.Cu, net GND

Commit message: interface-brain v1.0 complete
Parts:
- moved C37 105.4 mm to (146.4, 50.5)
- moved C47 97.8 mm to (162.9, 89.1), turned to 90 degrees
- moved C38 90.5 mm to (146.9, 85.8)
- moved C23 89.5 mm to (151.5, 72.9)
- moved C39 84.2 mm to (146.1, 92.8)
- moved C27 80.0 mm to (151.6, 88.1), turned to 0 degrees
- moved C26 77.3 mm to (151.6, 85.6), turned to 0 degrees
- moved C53 73.7 mm to (164.8, 99.9), turned to 0 degrees
- moved C44 71.4 mm to (165.4, 98.2), turned to -90 degrees
- moved C43 70.5 mm to (145.7, 84.1)
- moved C41 70.2 mm to (161.2, 50.2)
- moved C46 64.8 mm to (161.1, 93.5), turned to -90 degrees
- moved C25 62.1 mm to (147.0, 47.6)
- moved C42 56.4 mm to (162.9, 81.1), turned to -90 degrees
- moved C30 55.1 mm to (162.8, 77.6), turned to 90 degrees
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Connections:
- C23 pad 1: +3V3 -> GND
- C23 pad 2: GND -> +3V3
- J22 pad 1: GND -> +3V3
- J22 pad 3: +3V3 -> GND
- J23 pad 1: GND -> +3V3
- J23 pad 3: +3V3 -> GND
- J24 pad 1: GND -> +3V3
- J24 pad 3: +3V3 -> GND
- J25 pad 1: GND -> +3V3
- J25 pad 3: +3V3 -> GND
- J30 pad 1: GND -> +3V3
- J30 pad 3: +3V3 -> GND
- J31 pad 1: GND -> +3V3
- J31 pad 3: +3V3 -> GND
- J32 pad 1: GND -> +3V3
- J32 pad 3: +3V3 -> GND
- J33 pad 1: GND -> +3V3
- J33 pad 3: +3V3 -> GND
- U3 pad 46: +3V3 -> unconnected-(U3-Pad46)
Routing:
- net +5V: track 27.9 -> 623.1 mm, vias 1 -> 8
- net +3V3: track 11.2 -> 216.5 mm, vias 0 -> 2
- net GND: track 37.7 -> 92.6 mm, vias 0 -> 92
- net Net-(R12-Pad1): track 0.00 -> 20.4 mm, vias 0 -> 2
- net /BUTTON_13: track 174.0 -> 181.7 mm
- net /BUTTON_9: track 131.0 -> 134.3 mm
- net /ANALOG_8: track 52.5 -> 55.6 mm, vias 1 -> 2
- net /BUTTON_6: track 82.5 -> 85.4 mm
- net /LED8_OUT: track 0.00 -> 2.10 mm
- net /LED7_OUT: track 0.00 -> 1.99 mm
- net /BUTTON_2: track 114.2 -> 116.2 mm
- net /ANALOG_3: track 35.6 -> 37.5 mm
- net /ANALOG_7: track 90.9 -> 92.7 mm
- net /BUTTON_3: track 122.2 -> 124.0 mm
- net /BUTTON_4: track 118.9 -> 120.7 mm
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Other:
- board text added: "3V3"
- board text added: "5V"
- board text added: "CS"
- board text added: "G"
- board text added: "MISO"
- board text added: "MOSI"
- board text added: "PWR"
- board text added: "SCK"
- board text added: "interface-brain v1.0"

Commit message: interface-brain v1.1:
- Switch to serial-over-RS422 for comms with colordance-brain
- Add 12v supply + 5V SMPS
Parts:
- removed R8: 33, Resistor_SMD:R_0603_1608Metric
- added C54: 22uF, Capacitor_SMD:C_1206_3216Metric, B.Cu at (174.1, 72.7)
- added C55: 100nF, Capacitor_SMD:C_0402_1005Metric, B.Cu at (152.5, 97.0)
- added C56: 470uF, Capacitor_THT:CP_Radial_D10.0mm_P5.00mm, F.Cu at (169.3, 59.0)
- added C57: 1nF, Capacitor_SMD:C_0402_1005Metric, B.Cu at (145.4, 103.9)
- added C58: 100nF, Capacitor_SMD:C_0402_1005Metric, B.Cu at (176.0, 87.3)
- added C59: 10uF, Capacitor_SMD:C_0805_2012Metric, B.Cu at (171.7, 73.3)
- added C60: 100nF, Capacitor_SMD:C_0402_1005Metric, B.Cu at (175.9, 74.1)
- added C61: 10uF, Capacitor_SMD:C_0805_2012Metric, B.Cu at (152.4, 74.6)
- added D7: D_TVS_DATA, Diode_SMD:D_SMB, B.Cu at (156.8, 108.8)
- added D8: D_TVS_5V, Diode_SMD:D_SMB, B.Cu at (171.5, 67.5)
- added D9: D, Diode_SMD:D_SMA, B.Cu at (168.4, 77.5)
- added J40: RJ45, Connector_RJ:RJ45_Amphenol_54602-x08_Horizontal, F.Cu at (144.3, 108.3)
- added L1: 5.6uH, Inductor_SMD:L_Taiyo-Yuden_NR-60xx, B.Cu at (173.9, 78.8)
- added U4: ISL83490, Package_SO:SOIC-8_3.9x4.9mm_P1.27mm, B.Cu at (156.0, 98.7)
- added U5: AP3211, Package_TO_SOT_SMD:SOT-23-6, B.Cu at (173.7, 86.5)
- C5: value 100nF -> 470uF; footprint Capacitor_SMD:C_0402_1005Metric -> Capacitor_THT:CP_Radial_D10.0mm_P5.00mm; moved to F.Cu
- C6: footprint Capacitor_SMD:C_0603_1608Metric -> Capacitor_SMD:C_0805_2012Metric
- C7: value 470uF -> 10nF; footprint Capacitor_THT:CP_Radial_D10.0mm_P5.00mm -> Capacitor_SMD:C_0402_1005Metric; moved to B.Cu
- D1: value D_TVS_5V -> D_TVS_12V; footprint Diode_SMD:D_SOD-323 -> Diode_SMD:D_SMB
- D2: value D_TVS_5V -> SCHOTTKY; footprint Diode_SMD:D_SOD-323 -> Diode_SMD:D_SMA
- D3, D4, D5: value D_TVS_5V -> D_TVS_DATA; footprint Diode_SMD:D_SOD-323 -> Diode_SMD:D_SMB
- J1: value Conn_01x06 -> Anderson; footprint Homebrew:MiniPV_69167-X06XXX_1x06_P2.54mm_Polarized_Vertical -> Homebrew:Anderson_1336G1_right_angle_bottom_two
- R5: value 33 -> 11.5k
- R6: value 33 -> 2.21k
- R7: value 33 -> 120
- moved D6 69.2 mm to (171.0, 50.9)
- moved R25 69.2 mm to (172.6, 50.9)
- moved C7 30.5 mm to (171.3, 86.5), turned to -90 degrees
- moved R5 28.6 mm to (176.4, 84.5), turned to -90 degrees
- moved D2 25.6 mm to (168.5, 85.4)
- moved R6 25.1 mm to (174.0, 83.6), turned to 180 degrees
- moved C26 20.3 mm to (151.6, 65.3)
- moved C27 20.3 mm to (151.6, 67.8)
- moved J1 19.7 mm to (169.3, 105.0), turned to 180 degrees
- moved D1 19.2 mm to (169.7, 109.1), turned to 180 degrees
- moved C6 18.2 mm to (172.2, 90.7), turned to 180 degrees
- moved D3 15.8 mm to (139.8, 108.3), turned to -90 degrees
- moved R7 15.1 mm to (143.4, 105.4)
- moved H3 14.4 mm to (133.0, 108.4)
- moved C5 13.5 mm to (174.1, 97.3), turned to 180 degrees
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Connections:
- C5 pad 1: +5V -> +12V
- C6 pad 1: +5V -> +12V
- C7 pad 1: +5V -> Net-(C7-Pad1)
- C7 pad 2: GND -> Net-(C7-Pad2)
- D1 pad 1: GND -> +12V
- D1 pad 2: /SCK -> GND
- D2 pad 1: GND -> Net-(C7-Pad2)
- D2 pad 2: /MISO -> GND
- D3 pad 1: GND -> /SERIAL_Y
- D3 pad 2: /MOSI -> GND
- D4 pad 2: +5V -> /SERIAL_Z
- D5 pad 1: GND -> /SERIAL_B
- D5 pad 2: /CS -> GND
- J1 pad 1: GND -> +12V
- J1 pad 2: Net-(J1-Pad2) -> GND
- R5 pad 1: Net-(J1-Pad2) -> +5V
- R5 pad 2: /SCK -> Net-(R5-Pad2)
- R6 pad 1: Net-(J1-Pad3) -> Net-(R5-Pad2)
- R6 pad 2: /MISO -> GND
- R7 pad 1: Net-(J1-Pad4) -> /SERIAL_Y
- R7 pad 2: /MOSI -> Net-(C57-Pad1)
- U3 pad 12: /CS -> /BUTTON_3
- U3 pad 13: /MOSI -> /BUTTON_4
- U3 pad 14: /MISO -> unconnected-(U3-Pad14)
- U3 pad 20: /BUTTON_3 -> /SERIAL_IN
- U3 pad 21: /BUTTON_4 -> /SERIAL_OUT
- U3 pad 35: /SCK -> unconnected-(U3-Pad35)
Routing:
- net /CS: track 50.1 -> 0.00 mm, vias 1 -> 0
- net /SCK: track 47.0 -> 0.00 mm, vias 1 -> 0
- net /MOSI: track 45.7 -> 0.00 mm, vias 1 -> 0
- net /MISO: track 40.4 -> 0.00 mm, vias 1 -> 0
- net /SERIAL_Y: track 0.00 -> 31.5 mm, vias 0 -> 1
- net +12V: track 0.00 -> 25.4 mm
- net +3V3: track 216.5 -> 241.3 mm
- net /SERIAL_Z: track 0.00 -> 20.0 mm, vias 0 -> 1
- net /BUTTON_4: track 120.7 -> 136.8 mm, vias 2 -> 1
- net /SERIAL_IN: track 0.00 -> 16.1 mm, vias 0 -> 1
- net /SERIAL_B: track 0.00 -> 16.1 mm
- net /SERIAL_OUT: track 0.00 -> 15.3 mm, vias 0 -> 1
- net Net-(C7-Pad2): track 0.00 -> 13.9 mm, vias 0 -> 2
- net /BUTTON_13: track 181.7 -> 168.1 mm, vias 3 -> 1
- net Net-(C7-Pad1): track 0.00 -> 12.3 mm
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Other:
- board size 144 x 105 mm -> 154.5 x 105 mm
- board text added: "A"
- board text added: "B"
- board text added: "Y"
- board text added: "Z"
- board text added: "interface-brain v1.1"
- board text removed: "CS"
- board text removed: "MISO"
- board text removed: "MOSI"
- board text removed: "SCK"
- board text removed: "interface-brain v1.0"
