File: hardware/interface-brain/interface-brain.kicad_sch (KiCad schematic)
At the start: 156 parts, among them J10 Conn_01x03, J11 Conn_01x03, J12 Conn_01x03, J13 Conn_01x03, J14 Conn_01x03, J15 Conn_01x03, J16 Conn_01x03, J17 Conn_01x03, J19 Conn_01x02, J20 Conn_01x02, J21 Conn_01x02, J22 Conn_01x03, J23 Conn_01x03, J24 Conn_01x03, J25 Conn_01x03, J26 Conn_01x02, J27 Conn_01x02, J28 Conn_01x02, J29 Conn_01x02, J3 Conn_01x03, J30 Conn_01x03, J31 Conn_01x03, J32 Conn_01x03, J33 Conn_01x03, J34 Conn_01x02, J35 Conn_01x02, J36 Conn_01x02, J37 Conn_01x02, J38 Conn_01x02, J39 Conn_01x02, J4 Conn_01x03, J5 Conn_01x03, J6 Conn_01x03, J7 Conn_01x03, J8 Conn_01x03, J9 Conn_01x03, U2 SN74ACT244PWR

Commit message: Assign footprints and part numbers
Parts:
- C1, C10, C11, C12, C13, C14, C15, C16, C17, C18, C19, C2, C20, C21, C22, C23, C28, C29, C3, C30, C31, C32, C33, C34, C35, C4, C40, C41, C42, C43, C48, C49, C50, C51, C8, C9: value 100nF -> (none); footprint Capacitor_SMD:C_0402_1005Metric -> (none)
- C25, C26, C27, C36, C37, C38, C39, C44, C45, C46, C47, C52, C53: value 22nF -> (none); footprint Capacitor_SMD:C_0402_1005Metric -> (none)
- D2, D3, D4, D5: value D_TVS_5V -> (none); footprint Diode_SMD:D_SOD-323 -> (none)
- J1: MPN (none) -> 69167-106HLF
- J10, J11, J12, J13, J14, J15, J16, J17, J22, J23, J24, J25, J3, J30, J31, J32, J33, J4, J5, J6, J7, J8, J9: value Conn_01x03 -> (none); MPN (none) -> 69167-103HLF
- J18: MPN (none) -> 76384-302LF
- J19, J20, J21, J26, J27, J28, J29, J34, J35, J36, J37, J38, J39: value Conn_01x02 -> (none); MPN (none) -> 76384-302LF
- J2: MPN (none) -> 69167-103HLF
- R1, R2, R3, R4: value 10k -> (none); footprint Resistor_SMD:R_0603_1608Metric -> (none)
- R10, R11, R12, R13, R14, R15, R16, R18, R19, R20, R21, R22, R23, R24, R5, R6, R7, R8, R9: value 33 -> (none); footprint Resistor_SMD:R_0603_1608Metric -> (none)
- R27, R28, R29, R30, R31, R32, R33, R38, R39, R40, R41, R42, R43, R44, R45, R46, R47, R48, R49, R54, R55: value 1k -> (none); footprint Resistor_SMD:R_0603_1608Metric -> (none)
- R35, R36, R37, R50, R51, R52, R53: value DNP -> (none); footprint Resistor_SMD:R_0603_1608Metric -> (none)
- U1: LCSC (none) -> C6930
- U2: value SN74ACT244PWR -> (none); footprint SOP65P640X120-20N -> (none); LCSC (none) -> C6930
- U3: MPN (none) -> PPPC241LFBN-RC

Commit message: Continue interface brain layout
Parts:
- added H1, H2, H3, H4: (no value), symbol Mechanical:MountingHole
Connections:
- net BUTTON_3: now also U3.21 (29_TX7); no longer U3.6 (4_BCLK2)
- net BUTTON_6: now also U3.6 (4_BCLK2); no longer U3.21 (29_TX7)
- net LED10_OUT: now also J8.2 (Pin_2); no longer J11.2 (Pin_2)
- net LED10_SIG: now also U2.6 (1A3); no longer U2.4 (1A2)
- net LED11_SIG: now also U2.4 (1A2); no longer U2.6 (1A3)
- net LED12_OUT: now also J16.2 (Pin_2); no longer J13.2 (Pin_2)
- net LED12_SIG: now also U2.2 (1A1); no longer U2.8 (1A4)
- net LED13_OUT: now also J5.2 (Pin_2); no longer J14.2 (Pin_2)
- net LED14_OUT: now also J9.2 (Pin_2); no longer J15.2 (Pin_2)
- net LED15_OUT: now also J13.2 (Pin_2); no longer J16.2 (Pin_2)
- net LED1_SIG: now also U1.8 (1A4); no longer U1.2 (1A1)
- net LED2_OUT: now also J6.2 (Pin_2); no longer J3.2 (Pin_2)
- net LED2_SIG: now also U1.6 (1A3); no longer U1.4 (1A2)
- net LED3_OUT: now also J10.2 (Pin_2); no longer J4.2 (Pin_2)
- net LED3_SIG: now also U1.4 (1A2); no longer U1.6 (1A3)
- net LED4_OUT: now also J14.2 (Pin_2); no longer J5.2 (Pin_2)
- net LED4_SIG: now also U1.2 (1A1); no longer U1.8 (1A4)
- net LED5_OUT: now also J3.2 (Pin_2); no longer J6.2 (Pin_2)
- net LED7_OUT: now also J11.2 (Pin_2); no longer J8.2 (Pin_2)
- net LED8_OUT: now also J15.2 (Pin_2); no longer J9.2 (Pin_2)
- net LED9_OUT: now also J4.2 (Pin_2); no longer J10.2 (Pin_2)
- net LED9_SIG: now also U2.8 (1A4); no longer U2.2 (1A1)
- net at R21.1: now also U2.12 (1Y4); no longer U2.18 (1Y1)
- net at R17.1: now also U1.12 (1Y4); no longer U1.18 (1Y1)
- net at R22.1: now also U2.16 (1Y2); no longer U2.14 (1Y3)
- net at R13.1: now also U2.14 (1Y3); no longer U2.16 (1Y2)
- net at R9.1: now also U1.14 (1Y3); no longer U1.16 (1Y2)
- net at R10.1: now also U1.18 (1Y1); no longer U1.12 (1Y4)
- net at R18.1: now also U1.16 (1Y2); no longer U1.14 (1Y3)
- net at R14.1: now also U2.18 (1Y1); no longer U2.12 (1Y4)
Other:
- moved on the sheet: C13, R10, R13, R14, R17, R18, R21, R22, R9

Commit message: Interface brain layout almost done
Parts:
- C1, C10, C11, C12, C13, C14, C15, C16, C17, C18, C19, C2, C20, C21, C22, C23, C28, C29, C3, C30, C31, C32, C33, C34, C35, C4, C40, C41, C42, C43, C48, C49, C5, C50, C51, C8, C9: value (none) -> 100nF; footprint (none) -> Capacitor_SMD:C_0402_1005Metric
- C24, C25, C26, C27, C36, C37, C38, C39, C44, C45, C46, C47, C52, C53: value (none) -> 22nF; footprint (none) -> Capacitor_SMD:C_0402_1005Metric
- C6: value (none) -> 10uF; footprint (none) -> Capacitor_SMD:C_0603_1608Metric
- C7: value (none) -> 470uF; footprint (none) -> Capacitor_THT:CP_Radial_D10.0mm_P5.00mm
- D1, D2, D3, D4, D5: value (none) -> D_TVS_5V; footprint (none) -> Diode_SMD:D_SOD-323
- D6: value (none) -> LED; footprint (none) -> LED_SMD:LED_0603_1608Metric
- H1, H2, H3, H4: value (none) -> MountingHole; footprint (none) -> MountingHole:MountingHole_3.2mm_M3
- J1: value (none) -> Conn_01x06; footprint (none) -> Homebrew:MiniPV_69167-X06XXX_1x06_P2.54mm_Polarized_Vertical
- J10, J11, J12, J13, J14, J15, J16, J17, J2, J22, J23, J24, J25, J3, J30, J31, J32, J33, J4, J5, J6, J7, J8, J9: value (none) -> Conn_01x03; footprint (none) -> Homebrew:MiniPV_69167-X03XXX_1x03_P2.54mm_Polarized_Vertical
- J18, J19, J20, J21, J26, J27, J28, J29, J34, J35, J36, J37, J38, J39: value (none) -> Conn_01x02; footprint (none) -> Homebrew:MiniPV_76384-X02XX_1x02_P2.54mm_Vertical
- R1, R2, R25, R3, R4: value (none) -> 10k; footprint (none) -> Resistor_SMD:R_0603_1608Metric
- R10, R11, R12, R13, R14, R15, R16, R17, R18, R19, R20, R21, R22, R23, R24, R5, R6, R7, R8, R9: value (none) -> 33; footprint (none) -> Resistor_SMD:R_0603_1608Metric
- R26, R27, R28, R29, R30, R31, R32, R33, R38, R39, R40, R41, R42, R43, R44, R45, R46, R47, R48, R49, R54, R55: value (none) -> 1k; footprint (none) -> Resistor_SMD:R_0603_1608Metric
- R34, R35, R36, R37, R50, R51, R52, R53: value (none) -> DNP; footprint (none) -> Resistor_SMD:R_0603_1608Metric
- U1, U2: value (none) -> SN74ACT244PWR; footprint (none) -> Package_SO:TSSOP-20_4.4x6.5mm_P0.65mm
- U3: value (none) -> Teensy4.1; footprint (none) -> Homebrew:Teensy41_stripped
Connections:
- net ANALOG_2: now also U3.42 (20_A6_TX5_LRCLK1); no longer U3.31 (39_MISO1_OUT1A)
- net ANALOG_5: now also U3.18 (26_A12_MOSI1); no longer U3.42 (20_A6_TX5_LRCLK1)
- net ANALOG_7: now also U3.31 (39_MISO1_OUT1A); no longer U3.18 (26_A12_MOSI1)
- net BUTTON_10: now also U3.9 (7_RX2_OUT1A); no longer U3.26 (34_RX8)
- net BUTTON_14: now also U3.26 (34_RX8); no longer U3.9 (7_RX2_OUT1A)
- net BUTTON_3: now also U3.20 (28_RX7); no longer U3.21 (29_TX7)
- net BUTTON_4: now also U3.21 (29_TX7); no longer U3.7 (5_IN2)
- net BUTTON_5: now also U3.7 (5_IN2); no longer U3.20 (28_RX7)
- net LED11_SIG: now also U3.37 (15_A1_RX3_SPDIF_IN); no longer U3.44 (22_A8_CTX1)
- net LED12_SIG: now also U3.36 (14_A0_TX3_SPDIF_OUT); no longer U3.45 (23_A9_CRX1_MCLK1)
- net LED13_SIG: now also U3.11 (9_OUT1C); no longer U3.8 (6_OUT1D)
- net LED14_SIG: now also U3.16 (24_A10_TX6_SCL2); no longer U3.11 (9_OUT1C)
- net LED15_SIG: now also U3.17 (25_A11_RX6_SDA2); no longer U3.24 (32_OUT1B)
- net LED16_SIG: now also U3.24 (32_OUT1B); no longer U3.10 (8_TX2_IN1)
- net LED3_SIG: now also U3.8 (6_OUT1D); no longer U3.16 (24_A10_TX6_SCL2)
- net LED4_SIG: now also U3.10 (8_TX2_IN1); no longer U3.17 (25_A11_RX6_SDA2)
- net LED5_SIG: now also U3.45 (23_A9_CRX1_MCLK1); no longer U3.41 (19_A5_SCL)
- net LED6_SIG: now also U3.44 (22_A8_CTX1); no longer U3.40 (18_A4_SDA)
- net LED7_SIG: now also U3.41 (19_A5_SCL); no longer U3.36 (14_A0_TX3_SPDIF_OUT)
- net LED8_SIG: now also U3.40 (18_A4_SDA); no longer U3.37 (15_A1_RX3_SPDIF_IN)

Commit message: interface-brain v1.0 complete
Parts:
- C1, C10, C11, C12, C13, C14, C15, C16, C17, C18, C19, C2, C20, C21, C22, C23, C28, C29, C3, C30, C31, C32, C33, C34, C35, C4, C40, C41, C42, C43, C48, C49, C5, C50, C51, C8, C9: value 100nF -> (none); footprint Capacitor_SMD:C_0402_1005Metric -> (none)
- C24, C25, C26, C27, C36, C37, C38, C39, C44, C45, C46, C47, C52, C53: value 22nF -> (none); footprint Capacitor_SMD:C_0402_1005Metric -> (none)
- C6: value 10uF -> (none); footprint Capacitor_SMD:C_0603_1608Metric -> (none)
- C7: value 470uF -> (none); footprint Capacitor_THT:CP_Radial_D10.0mm_P5.00mm -> (none)
- D1, D2, D3, D4, D5: value D_TVS_5V -> (none); footprint Diode_SMD:D_SOD-323 -> (none)
- D6: value LED -> (none); footprint LED_SMD:LED_0603_1608Metric -> (none)
- H1, H2, H3, H4: value MountingHole -> (none); footprint MountingHole:MountingHole_3.2mm_M3 -> (none)
- J1: value Conn_01x06 -> (none); footprint Homebrew:MiniPV_69167-X06XXX_1x06_P2.54mm_Polarized_Vertical -> (none)
- J10, J11, J12, J13, J14, J15, J16, J17, J2, J22, J23, J24, J25, J3, J30, J31, J32, J33, J4, J5, J6, J7, J8, J9: value Conn_01x03 -> (none); footprint Homebrew:MiniPV_69167-X03XXX_1x03_P2.54mm_Polarized_Vertical -> (none)
- J18, J19, J20, J21, J26, J27, J28, J29, J34, J35, J36, J37, J38, J39: value Conn_01x02 -> (none); footprint Homebrew:MiniPV_76384-X02XX_1x02_P2.54mm_Vertical -> (none)
- R1, R2, R25, R3, R4: value 10k -> (none); footprint Resistor_SMD:R_0603_1608Metric -> (none)
- R10, R11, R12, R13, R14, R15, R16, R17, R18, R19, R20, R21, R22, R23, R24, R5, R6, R7, R8, R9: value 33 -> (none); footprint Resistor_SMD:R_0603_1608Metric -> (none)
- R26, R27, R28, R29, R30, R31, R32, R33, R38, R39, R40, R41, R42, R43, R44, R45, R46, R47, R48, R49, R54, R55: value 1k -> (none); footprint Resistor_SMD:R_0603_1608Metric -> (none)
- R34, R35, R36, R37, R50, R51, R52, R53: value DNP -> (none); footprint Resistor_SMD:R_0603_1608Metric -> (none)
- U1, U2: value SN74ACT244PWR -> (none); footprint Package_SO:TSSOP-20_4.4x6.5mm_P0.65mm -> (none)
- U3: value Teensy4.1 -> (none); footprint Homebrew:Teensy41_stripped -> (none)
Connections:
- net +3V3: now also C23.2, J22.1 (Pin_1), J23.1 (Pin_1), J24.1 (Pin_1), J25.1 (Pin_1), J30.1 (Pin_1), J31.1 (Pin_1), J32.1 (Pin_1), J33.1 (Pin_1); no longer C23.1, J22.3 (Pin_3), J23.3 (Pin_3), J24.3 (Pin_3), J25.3 (Pin_3), J30.3 (Pin_3), J31.3 (Pin_3), J32.3 (Pin_3), J33.3 (Pin_3), U3.46 (3V3)
- net GND: now also C23.1, J22.3 (Pin_3), J23.3 (Pin_3), J24.3 (Pin_3), J25.3 (Pin_3), J30.3 (Pin_3), J31.3 (Pin_3), J32.3 (Pin_3), J33.3 (Pin_3); no longer C23.2, J22.1 (Pin_1), J23.1 (Pin_1), J24.1 (Pin_1), J25.1 (Pin_1), J30.1 (Pin_1), J31.1 (Pin_1), J32.1 (Pin_1), J33.1 (Pin_1)
- no-connect marks 19 -> 20
Other:
- moved on the sheet: C23, J22, J23, J24, J25, J30, J31, J32, J33

Commit message: Update interface-brain schematic
Parts:
- removed C5, C6: (no value), symbol Device:C
- removed C7: (no value), symbol Device:C_Polarized
- removed D1, D2: (no value), symbol Device:D_TVS
- removed J1: (no value), symbol Connector_Generic:Conn_01x06
- removed R5, R6, R8: (no value), symbol Device:R
- added C55: 100nF, Capacitor_SMD:C_0402_1005Metric, symbol Device:C
- added C57: 1nF, Capacitor_SMD:C_0402_1005Metric, symbol Device:C
- added C61: 10uF, Capacitor_SMD:C_0805_2012Metric, symbol Device:C
- added D7: D_TVS_DATA, Diode_SMD:D_SMB, symbol Device:D_TVS
- added J40: RJ45, Connector_RJ:RJ45_Amphenol_54602-x08_Horizontal, symbol Connector:RJ45
- added U4: ISL83490, Package_SO:SOIC-8_3.9x4.9mm_P1.27mm, symbol homebrew:ISL83490
- C1, C10, C11, C12, C13, C14, C15, C16, C17, C18, C19, C2, C20, C21, C22, C23, C28, C29, C3, C30, C31, C32, C33, C34, C35, C4, C40, C41, C42, C43, C48, C49, C50, C51, C8, C9: value (none) -> 100nF; footprint (none) -> Capacitor_SMD:C_0402_1005Metric
- C24, C25, C26, C27, C36, C37, C38, C39, C44, C45, C46, C47, C52, C53: value (none) -> 22nF; footprint (none) -> Capacitor_SMD:C_0402_1005Metric
- D3, D4, D5: value (none) -> D_TVS_DATA; footprint (none) -> Diode_SMD:D_SMB; LCSC C182013 -> (none); MPN (none) -> SMBJ6.0CD-M3/H
- D6: value (none) -> LED; footprint (none) -> LED_SMD:LED_0603_1608Metric
- H1, H2, H3, H4: value (none) -> MountingHole; footprint (none) -> MountingHole:MountingHole_3.2mm_M3
- J10, J11, J12, J13, J14, J15, J16, J17, J2, J22, J23, J24, J25, J3, J30, J31, J32, J33, J4, J5, J6, J7, J8, J9: value (none) -> Conn_01x03; footprint (none) -> Homebrew:MiniPV_69167-X03XXX_1x03_P2.54mm_Polarized_Vertical
- J18, J19, J20, J21, J26, J27, J28, J29, J34, J35, J36, J37, J38, J39: value (none) -> Conn_01x02; footprint (none) -> Homebrew:MiniPV_76384-X02XX_1x02_P2.54mm_Vertical
- R1, R2, R25, R3, R4: value (none) -> 10k; footprint (none) -> Resistor_SMD:R_0603_1608Metric
- R10, R11, R12, R13, R14, R15, R16, R17, R18, R19, R20, R21, R22, R23, R24, R9: value (none) -> 33; footprint (none) -> Resistor_SMD:R_0603_1608Metric
- R26, R27, R28, R29, R30, R31, R32, R33, R38, R39, R40, R41, R42, R43, R44, R45, R46, R47, R48, R49, R54, R55: value (none) -> 1k; footprint (none) -> Resistor_SMD:R_0603_1608Metric
- R34, R35, R36, R37, R50, R51, R52, R53: value (none) -> DNP; footprint (none) -> Resistor_SMD:R_0603_1608Metric
- R7: value (none) -> 120; footprint (none) -> Resistor_SMD:R_0603_1608Metric; LCSC C23140 -> C25808
- U1, U2: value (none) -> SN74ACT244PWR; footprint (none) -> Package_SO:TSSOP-20_4.4x6.5mm_P0.65mm
- U3: value (none) -> Teensy4.1; footprint (none) -> Homebrew:Teensy41_stripped
Connections:
- net +3V3: now also C55.1, C61.2, U4.1 (VCC)
- net +5V: no longer D4.2 (A2)
- net BUTTON_3: now also U3.12 (10_CS_MQSR); no longer U3.20 (28_RX7)
- net BUTTON_4: now also U3.13 (11_MOSI_CTX1); no longer U3.21 (29_TX7)
- net GND: now also D3.2 (A2), D5.2 (A2), C55.2, C61.1, D7.1 (A1), J40.3, J40.4, J40.5, J40.6, U4.4 (GND); no longer D3.1 (A1), D5.1 (A1)
- net SERIAL_Y: now reaches R7.1
- net SERIAL_Y: now also D3.1 (A1), J40.1, U4.5 (Y)
- removed net CS: D5.2 (A2), U3.12 (10_CS_MQSR)
- net MISO: no longer names the net of U3.14 (12_MISO_MQSL)
- removed net MOSI: D3.2 (A2), R7.2, U3.13 (11_MOSI_CTX1)
- net SCK: no longer names the net of U3.35 (13_SCK_LED)
- new net: C57.1, R7.2
- new net SERIAL_A: D7.2 (A2), J40.8, U4.8 (A)
- new net SERIAL_B: D5.1 (A1), J40.7, U4.7 (B)
- new net SERIAL_IN: U3.20 (28_RX7), U4.2 (RO)
- new net SERIAL_OUT: U3.21 (29_TX7), U4.3 (DI)
- new net SERIAL_Z: C57.2, D4.2 (A2), J40.2, U4.6 (Z)
- no-connect marks 20 -> 22
Other:
- added sheet 5v_smps (5v_smps.kicad_sch)
- moved on the sheet: C1, C10, C11, C12, C13, C14, C15, C16, C17, C18, C19, C2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

Commit message: interface-brain v1.1:
- Switch to serial-over-RS422 for comms with colordance-brain
- Add 12v supply + 5V SMPS
Parts:
- R7: LCSC C25808 -> C22787
Changed lines of the file:
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@@
       (effects (font (size 1.27 1.27)) hide)
     )
-    (property "LCSC" "C25808" (id 4) (at 469.9 40.64 0)
+    (property "LCSC" "C22787" (id 4) (at 469.9 40.64 0)
       (effects (font (size 1.27 1.27)) hide)
     )
@@
     )
     (path "/d842a1be-ffa0-45ce-984e-638142f4a2db/f575f0cf-b65d-4375-92ee-5a29c03e83d6"
-      (reference "J1") (unit 1) (value "Anderson") (footprint "homebrew:Anderson_1336G1_right_angle_bottom_two")
+      (reference "J1") (unit 1) (value "Anderson") (footprint "Homebrew:Anderson_1336G1_right_angle_bottom_two")
     )
     (path "/e22bb1c2-6aa0-48f7-ad07-4af57f61927c"
